File: arduino_can_bus_shield_v2/arduino_can_bus_shield_v2.kicad_pcb (KiCad board)
At the start: 2 copper layers, 26 parts, among them J1 molex_3.0, J2 molex_3.0, J3 MPU9250, J4 OLED, J5 UART2, J6 Encoder 1, J7 Encoder 0, SW1 SW_DIP_x04, SW2 User, SW3 User, U1 MCP2551-I-SN, U2 MCP2515-xST, Y1 16MHz

Commit message: Add files via upload
Parts:
- added P1: Power, Socket_Arduino_Uno:Socket_Strip_Arduino_1x08, F.Cu at (106.7, 160.0)
- added P2: Analog, Socket_Arduino_Uno:Socket_Strip_Arduino_1x06, F.Cu at (129.5, 160.0)
- added P3: Digital, Socket_Arduino_Uno:Socket_Strip_Arduino_1x10, F.Cu at (97.5, 111.8)
- added P4: Digital, Socket_Arduino_Uno:Socket_Strip_Arduino_1x08, F.Cu at (124.5, 111.8)
- added P5: CONN_01X01, Socket_Arduino_Uno:Arduino_1pin, F.Cu at (92.7, 160.0)
- added P6: CONN_01X01, Socket_Arduino_Uno:Arduino_1pin, F.Cu at (144.8, 154.9)
- added P7: CONN_01X01, Socket_Arduino_Uno:Arduino_1pin, F.Cu at (94.0, 111.8)
- added P8: CONN_01X01, Socket_Arduino_Uno:Arduino_1pin, F.Cu at (144.8, 127.0)
- C1, C2, C3, C4, J1, J2, JP1, JP2, R1, R3, R5, U1, U2: moved to B.Cu
- moved D1 116.2 mm to (99.1, 160.0)
- moved J3 102.4 mm to (91.4, 144.3), turned to 180 degrees
- moved R2 98.3 mm to (122.4, 156.0), turned to 180 degrees
- moved R6 93.4 mm to (103.0, 160.0), turned to -90 degrees
- moved J6 89.6 mm to (107.9, 153.7), turned to -90 degrees
- moved J7 85.3 mm to (107.9, 149.9), turned to -90 degrees
- moved J1 75.3 mm to (135.5, 147.3), turned to 90 degrees
- moved SW3 74.3 mm to (131.2, 136.1)
- moved J5 72.5 mm to (138.7, 136.6), turned to 180 degrees
- moved U2 69.2 mm to (111.1, 127.3), turned to 90 degrees
- moved R1 67.8 mm to (105.5, 144.8), turned to 180 degrees
- moved SW1 63.5 mm to (120.6, 143.8)
- moved R4 62.9 mm to (128.1, 124.5)
- moved JP2 61.6 mm to (116.2, 154.6), turned to 90 degrees
- moved U1 57.8 mm to (111.4, 141.6)
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Connections:
- C2 pad 1: +5V -> /can_enable
Other:
- board outline added: 58.4 x 53.3 mm
- board text added: "1"
