File: arduino_can_bus_shield_v2/arduino_can_bus_shield_v2.kicad_sch (KiCad schematic)
At the start: 30 parts, among them J1 molex_3.0, J2 molex_3.0, J3 MPU9250, J4 OLED, J5 UART2, J6 Encoder 1, J7 Encoder 0, P1 Power, P2 Analog, P3 Digital, P4 Digital, SW1 SW_DIP_x04, SW2 User, SW3 User, U1 MCP2551-I-SN, U2 MCP2515-xST, Y1 16MHz

Commit message: Add files via upload
Parts:
- added P5, P6, P7, P8: CONN_01X01, Socket_Arduino_Uno:Arduino_1pin, symbol Connector_Generic:Conn_01x01
- JP1: footprint (none) -> Jumper:SolderJumper-3_P1.3mm_Open_Pad1.0x1.5mm_NumberLabels
Connections:
- net SCL is gone; now on net A5(SCL): P3.1 (Pin_1)
- net SDA is gone; now on net A4(SDA): P3.2 (Pin_2)
- net +5V: no longer C2.1
- net can_enable: now also C2.1
- no-connect marks 17 -> 21
Other:
- note added: "Holes"
- note added: "Shield for Arduino that uses the same pin disposition like "Uno" board Rev 3."
- note removed: "Arduino Uno pinout"
